Commit message: Add accurate arena model to robot simulation

File: ros/catkin_ws/src/megabot_description/urdf/megabot.urdf (robot description, URDF)
Before this commit: robot test_model, 2 links, 1 joints
Links:
- link base_link: geometry collision box size=0.46 0.46 0.46; visual box size=0.46 0.46 0.46

File: ros/catkin_ws/src/megabot_description/urdf/tennis_ball.urdf (robot description, URDF)
Before this commit: robot tennis_ball, 1 links, 0 joints
Links:
- link ball: geometry collision sphere radius=0.033; visual sphere radius=0.033

Commit message: Increase realism by adding textures and bouncing ball

File: ros/catkin_ws/src/megabot_description/urdf/megabot.urdf (robot description, URDF)
Before this commit: robot test_model, 2 links, 1 joints
Joints:
- joint base_link_joint: origin xyz=0.0 0 0.5 rpy=0 0 0 -> xyz=0.0 0 0.23 rpy=0 0 0
