Commit message: Add more accurate robot model with camera

File: ros/catkin_ws/src/megabot_description/urdf/wheel.urdf.xacro (robot description, xacro)
@@ -1,4 +1,5 @@
 <?xml version="1.0"?>
 <robot xmlns:xacro="http://ros.org/wiki/xacro" name="megabot_wheel">
+	<!-- Define macro for wheel -->
 	<xacro:macro name="megabot_wheel" params="wheel_prefix *joint_pose">
 		<link name="${wheel_prefix}_wheel_link">
@@ -9,7 +10,7 @@
 			</inertial>
 			<visual>
-				<origin xyz="0 0 0" rpy="0 0 0" />
+				<origin xyz="0 0 0" rpy="${M_PI/2} 0 0" />
 				<geometry>
-					<mesh filename="package://husky_description/meshes/wheel.dae" />
+					<cylinder length="${wheel_length}" radius="${wheel_radius}" />
 				</geometry>
 			</visual>
@@ -28,5 +29,5 @@
 			<fdir1 value="1 0 0"/>
 		</gazebo>
-		<joint name="${wheel_prefix}_wheel" type="continuous">
+		<joint name="${wheel_prefix}_wheel" type="fixed">
 			<parent link="base_link"/>
 			<child link="${wheel_prefix}_wheel_link"/>
@@ -34,13 +35,4 @@
 			<axis xyz="0 1 0" rpy="0 0 0" />
 		</joint>
-		<transmission name="${wheel_prefix}_wheel_trans" type="SimpleTransmission">
-			<type>transmission_interface/SimpleTransmission</type>
-			<actuator name="${wheel_prefix}_wheel_motor">
-				<mechanicalReduction>1</mechanicalReduction>
-			</actuator>
-			<joint name="${wheel_prefix}_wheel">
-				<hardwareInterface>hardware_interface/VelocityJointInterface</hardwareInterface>
-			</joint>
-		</transmission>
 	</xacro:macro>
 </robot>
