Commit message: Add rangefinders to be used in localisation maybe

File: ros/catkin_ws/src/megabot/urdf/megabot.urdf.xacro (robot description, xacro)
@@ -4,4 +4,5 @@
   <xacro:include filename="$(find megabot)/urdf/wheel.urdf.xacro" />
   <xacro:include filename="$(find megabot)/urdf/camera.urdf.xacro" />
+  <xacro:include filename="$(find hector_sensors_description)/urdf/sonar_sensor.urdf.xacro" />
   <!-- Global constants -->
   <xacro:property name="M_PI" value="3.14159"/>
@@ -88,4 +89,21 @@
   <!-- Add camera via macros -->
   <xacro:megabot_camera />
+  <xacro:property name="sonar_ur" value="25.0"/>
+  <xacro:property name="sonar_min_rng" value="0.1"/>
+  <xacro:property name="sonar_max_rng" value="0.8"/>
+  <xacro:property name="sonar_fov" value="0.1"/>
+  <xacro:property name="sonar_rc" value="5"/>
+  <xacro:sonar_sensor name="sonar_front" parent="base_plate" ros_topic="sonar_front" update_rate="${sonar_ur}" min_range="${sonar_min_rng}" max_range="${sonar_max_rng}" field_of_view="${sonar_fov}" ray_count="${sonar_rc}">
+    <origin xyz="${wheelbase/2} 0 0" rpy="0 0 0"/>
+  </xacro:sonar_sensor>
+  <xacro:sonar_sensor name="sonar_left" parent="base_plate" ros_topic="sonar_left" update_rate="${sonar_ur}" min_range="${sonar_min_rng}" max_range="${sonar_max_rng}" field_of_view="${sonar_fov}" ray_count="${sonar_rc}">
+    <origin xyz="0 ${track/2} 0" rpy="0 0 ${M_PI/2}"/>
+  </xacro:sonar_sensor>
+  <xacro:sonar_sensor name="sonar_right" parent="base_plate" ros_topic="sonar_right" update_rate="${sonar_ur}" min_range="${sonar_min_rng}" max_range="${sonar_max_rng}" field_of_view="${sonar_fov}" ray_count="${sonar_rc}">
+    <origin xyz="0 -${track/2} 0" rpy="0 0 -${M_PI/2}"/>
+  </xacro:sonar_sensor>
+  <xacro:sonar_sensor name="sonar_back" parent="base_plate" ros_topic="sonar_back" update_rate="${sonar_ur}" min_range="${sonar_min_rng}" max_range="${sonar_max_rng}" field_of_view="${sonar_fov}" ray_count="${sonar_rc}">
+    <origin xyz="-${wheelbase/2} 0 0" rpy="0 0 ${M_PI}"/>
+  </xacro:sonar_sensor>
   <!-- Set method of motion control in Gazebo -->
   <gazebo>
@@ -97,4 +115,16 @@
       <robotBaseFrame>base_footprint</robotBaseFrame>
     </plugin>
+    <plugin name="magnetometer" filename="libhector_gazebo_ros_magnetic.so">
+      <updateRate>20.0</updateRate>
+      <robotNamespace>megabot</robotNamespace>
+      <bodyName>base_footprint</bodyName>
+      <drift>0 0 0</drift>
+      <driftFrequency>0 0 0</driftFrequency>
+      <gaussianNoise>0 0 0</gaussianNoise>
+      <!-- <referenceHeading>0.0</referenceHeading> -->
+      <!-- <declination>0</declination> -->
+      <!-- <inclination>0</inclination> -->
+      <!-- <offset>0 0 0</offset> -->
+    </plugin>
   </gazebo>
 </robot>

Commit message: Ball localisation working on real robot

File: ros/catkin_ws/src/megabot/urdf/megabot.urdf.xacro (robot description, xacro)
@@ -83,8 +83,8 @@
   </xacro:megabot_wheel>
   <!-- Camera parameters -->
-  <xacro:property name="camera_size" value="0.03" /> <!-- Size of square 'camera' box -->
-  <xacro:property name="camera_front_offset" value="0.1" /> <!-- Size of square 'camera' box -->
-  <xacro:property name="camera_height" value="0.4" /> <!-- Size of square 'camera' box -->
-  <xacro:property name="camera_pitch" value="0.8" /> <!-- Size of square 'camera' box -->
+  <xacro:property name="camera_size" value="0.03" />
+  <xacro:property name="camera_front_offset" value="0.185" />
+  <xacro:property name="camera_height" value="0.43" />
+  <xacro:property name="camera_pitch" value="1.22" />
   <!-- Add camera via macros -->
   <xacro:megabot_camera />

Commit message: Add robot based odom and inital draft of master state machine

File: ros/catkin_ws/src/megabot/urdf/megabot.urdf.xacro (robot description, xacro)
@@ -61,4 +61,42 @@
     <parent link="base_link"/>
     <child link="base_plate" />
+  </joint>
+  <link name="right_grabber">
+    <inertial>
+      <mass value="50" />
+      <origin xyz="0 0 0" />
+      <inertia ixx="50.0" ixy="0.0" ixz="0.0"
+        iyy="50.0" iyz="0.0"
+        izz="50.0" />
+    </inertial>
+    <visual>
+      <geometry>
+        <sphere size="0.3" />
+      </geometry>
+    </visual>
+  </link>
+  <joint name="right_grabber_joint" type="fixed">
+    <origin xyz="0.239 -0.067 0.03" rpy="0 0 0" />
+    <parent link="base_footprint"/>
+    <child link="right_grabber" />
+  </joint>
+  <link name="left_grabber">
+    <inertial>
+      <mass value="50" />
+      <origin xyz="0 0 0" />
+      <inertia ixx="50.0" ixy="0.0" ixz="0.0"
+        iyy="50.0" iyz="0.0"
+        izz="50.0" />
+    </inertial>
+    <visual>
+      <geometry>
+        <sphere size="0.3" />
+      </geometry>
+    </visual>
+  </link>
+  <joint name="left_grabber_joint" type="fixed">
+    <origin xyz="0.239 0.067 0.03" rpy="0 0 0" />
+    <parent link="base_footprint"/>
+    <child link="left_grabber" />
   </joint>
   <!-- Wheel parameters -->

Commit message: State machine for initial portion working

File: ros/catkin_ws/src/megabot/urdf/megabot.urdf.xacro (robot description, xacro)
@@ -72,5 +72,5 @@
     <visual>
       <geometry>
-        <sphere size="0.3" />
+        <sphere radius="0.033" />
       </geometry>
     </visual>
@@ -91,10 +91,10 @@
     <visual>
       <geometry>
-        <sphere size="0.3" />
+        <sphere radius="0.033" />
       </geometry>
     </visual>
   </link>
   <joint name="left_grabber_joint" type="fixed">
-    <origin xyz="0.239 0.067 0.03" rpy="0 0 0" />
+    <origin xyz="0.231 0.039 0.03" rpy="0 0 0" />
     <parent link="base_footprint"/>
     <child link="left_grabber" />

Commit message: Add grabber stage locations

File: ros/catkin_ws/src/megabot/urdf/megabot.urdf.xacro (robot description, xacro)
@@ -77,7 +77,26 @@
   </link>
   <joint name="right_grabber_joint" type="fixed">
-    <origin xyz="0.239 -0.067 0.03" rpy="0 0 0" />
+    <origin xyz="0.231 -0.039 0.03" rpy="0 0 0" />
     <parent link="base_footprint"/>
     <child link="right_grabber" />
+  </joint>
+  <link name="right_grabber_stage">
+    <inertial>
+      <mass value="50" />
+      <origin xyz="0 0 0" />
+      <inertia ixx="50.0" ixy="0.0" ixz="0.0"
+        iyy="50.0" iyz="0.0"
+        izz="50.0" />
+    </inertial>
+    <visual>
+      <geometry>
+        <sphere radius="0.01" />
+      </geometry>
+    </visual>
+  </link>
+  <joint name="right_grabber_stage_joint" type="fixed">
+    <origin xyz="0.1 0.0 0.03" rpy="0 0 0" />
+    <parent link="right_grabber"/>
+    <child link="right_grabber_stage" />
   </joint>
   <link name="left_grabber">
@@ -99,4 +118,23 @@
     <parent link="base_footprint"/>
     <child link="left_grabber" />
+  </joint>
+  <link name="left_grabber_stage">
+    <inertial>
+      <mass value="50" />
+      <origin xyz="0 0 0" />
+      <inertia ixx="50.0" ixy="0.0" ixz="0.0"
+        iyy="50.0" iyz="0.0"
+        izz="50.0" />
+    </inertial>
+    <visual>
+      <geometry>
+        <sphere radius="0.01" />
+      </geometry>
+    </visual>
+  </link>
+  <joint name="left_grabber_stage_joint" type="fixed">
+    <origin xyz="0.1 0.0 0.03" rpy="0 0 0" />
+    <parent link="left_grabber"/>
+    <child link="left_grabber_stage" />
   </joint>
   <!-- Wheel parameters -->

Commit message: Update master state machine for distance limit on moves

File: ros/catkin_ws/src/megabot/urdf/megabot.urdf.xacro (robot description, xacro)
@@ -77,5 +77,5 @@
   </link>
   <joint name="right_grabber_joint" type="fixed">
-    <origin xyz="0.231 -0.039 0.03" rpy="0 0 0" />
+    <origin xyz="0.231 -0.059 0.03" rpy="0 0 0" />
     <parent link="base_footprint"/>
     <child link="right_grabber" />
@@ -115,5 +115,5 @@
   </link>
   <joint name="left_grabber_joint" type="fixed">
-    <origin xyz="0.231 0.039 0.03" rpy="0 0 0" />
+    <origin xyz="0.231 0.059 0.03" rpy="0 0 0" />
     <parent link="base_footprint"/>
     <child link="left_grabber" />

Commit message: Improve camera location values

File: ros/catkin_ws/src/megabot/urdf/megabot.urdf.xacro (robot description, xacro)
@@ -160,5 +160,5 @@
   <!-- Camera parameters -->
   <xacro:property name="camera_size" value="0.03" />
-  <xacro:property name="camera_front_offset" value="0.185" />
+  <xacro:property name="camera_front_offset" value="0.165" />
   <xacro:property name="camera_height" value="0.43" />
   <xacro:property name="camera_pitch" value="1.22" />

Commit message: Update parameters

File: ros/catkin_ws/src/megabot/urdf/megabot.urdf.xacro (robot description, xacro)
@@ -77,5 +77,5 @@
   </link>
   <joint name="right_grabber_joint" type="fixed">
-    <origin xyz="0.231 -0.059 0.03" rpy="0 0 0" />
+    <origin xyz="0.221 -0.059 0.03" rpy="0 0 0" />
     <parent link="base_footprint"/>
     <child link="right_grabber" />
@@ -115,5 +115,5 @@
   </link>
   <joint name="left_grabber_joint" type="fixed">
-    <origin xyz="0.231 0.059 0.03" rpy="0 0 0" />
+    <origin xyz="0.221 0.059 0.03" rpy="0 0 0" />
     <parent link="base_footprint"/>
     <child link="left_grabber" />
